File: NewSub2023/2023PowerDistro/2023PowerDistro.kicad_pcb (KiCad board)
At the start: 2 copper layers, 36 x 18.1 mm, 29 parts, among them J1 Battery 1 Input, J2 Battery 2 Input, SW1 Power Switch

Commit message: Added traces to new power distro
Parts:
- moved D1 358.0 mm to (528.6, 102.3)
- moved D2 358.0 mm to (528.6, 105.9)
- moved C1 358.0 mm to (522.7, 103.8)
- moved C2 358.0 mm to (522.7, 110.4)
- moved C3 358.0 mm to (522.7, 117.0)
- moved F1 349.2 mm to (442.0, 190.5)
- moved Us8 348.8 mm to (489.4, 315.2)
- moved Us2 347.6 mm to (489.4, 216.1)
- moved Us4 347.6 mm to (489.4, 249.1)
- moved Us6 347.6 mm to (489.4, 282.1)
- moved Us5 344.7 mm to (400.5, 266.3)
- moved Us7 343.7 mm to (400.5, 298.7)
- moved Us9 343.7 mm to (400.5, 331.7)
- moved J10 340.1 mm to (330.6, 345.3)
- moved J5 340.1 mm to (330.7, 263.1)
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Connections:
- J10 pad 2: Net-(J10-B) -> Net-(J10-C)
Routing:
- net Net-(J9-C): track 0.00 -> 190.9 mm
- net Net-(J3-C): track 0.00 -> 109.4 mm
- net Net-(J5-C): track 0.00 -> 109.4 mm
- net Net-(J7-A): track 0.00 -> 109.4 mm
- net Net-(J7-C): track 0.00 -> 109.4 mm
- net Net-(J9-A): track 0.00 -> 109.3 mm
- net Net-(J5-A): track 0.00 -> 109.3 mm
- net Net-(J3-A): track 0.00 -> 109.3 mm
- net Net-(J7-B): track 0.00 -> 108.6 mm
- net Net-(J5-B): track 0.00 -> 108.5 mm
- net Net-(J3-B): track 0.00 -> 108.5 mm
- net Net-(J9-B): track 0.00 -> 108.5 mm
- net Net-(J4-B): track 0.00 -> 26.0 mm
- net Net-(J8-A): track 0.00 -> 20.6 mm
- net Net-(J6-A): track 0.00 -> 20.6 mm
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Other:
- board size 36 x 18.1 mm -> 235 x 215 mm
