File: 2024/PowerDistro/PowerDistro.kicad_pcb (KiCad board)
At the start: 4 copper layers, 235 x 285 mm, 47 parts, among them J1 10159560-A00221RLF, J2 AMPHENOL_10159560-A00221RLF, J3 AMPHENOL_10159560-A00221RLF, J4 AMPHENOL_10159560-A00221RLF, J5 AMPHENOL_10159560-A00221RLF, J6 AMPHENOL_10159560-A00221RLF, J7 AMPHENOL_10159560-A00221RLF, J8 AMPHENOL_10159560-A00221RLF, U1 TSSOP28

Commit message: Added motor controller squares
Parts:
- removed H2, H3, H4: M2.5, MountingHole:MountingHole_2.7mm_M2.5_ISO7380
- removed the J5 at (26.0, 71.2)
- added H1: M2.5, MountingHole:MountingHole_2.7mm_M2.5_ISO7380, F.Cu at (90.8, -16.2)
- added H1: M2.5, MountingHole:MountingHole_2.7mm_M2.5_ISO7380, F.Cu at (90.8, 33.8)
- added H1: M2.5, MountingHole:MountingHole_2.7mm_M2.5_ISO7380, F.Cu at (307.2, 22.7)
- added H1: M2.5, MountingHole:MountingHole_2.7mm_M2.5_ISO7380, F.Cu at (90.8, 83.8)
- added H1: M2.5, MountingHole:MountingHole_2.7mm_M2.5_ISO7380, F.Cu at (231.2, 22.2)
- added H1: M2.5, MountingHole:MountingHole_2.7mm_M2.5_ISO7380, F.Cu at (307.7, 122.2)
- added H1: M2.5, MountingHole:MountingHole_2.7mm_M2.5_ISO7380, F.Cu at (231.7, 122.6)
- added J1: 10159560-A00221RLF, PowerDistroFootprints:AMPHENOL_10159560-A00221RLF, F.Cu at (248.7, 103.2)
- J2, J3, J4, J6, J7, J8: value AMPHENOL_10159560-A00221RLF -> 10159560-A00221RLF
- J5: renamed from J1; footprint EasyBLDC:AMPHENOL_10159560-A00221RLF -> PowerDistroFootprints:AMPHENOL_10159560-A00221RLF
- JP4: value JST_SM06B-GHS-TB_LF__SN_ -> SM06B-GHS-TB_LF__SN_
- U1: value TSSOP28 -> PCA9685
- moved J6 219.8 mm to (248.2, 3.66)
- moved R8 193.5 mm to (239.2, -37.0), turned to 0 degrees
- moved R10 192.6 mm to (230.4, -31.6)
- moved R7 192.6 mm to (246.8, -45.6)
- moved JP4 192.6 mm to (234.6, -39.1)
- moved LED1 192.6 mm to (229.6, -34.8)
- moved U1 192.6 mm to (246.7, -39.5)
- moved R9 192.3 mm to (239.2, -39.5), turned to 180 degrees
- moved R11 191.6 mm to (247.8, -27.5), turned to 90 degrees
- moved R12 191.6 mm to (245.3, -27.5), turned to 90 degrees
- moved R13 191.6 mm to (242.8, -27.5), turned to 90 degrees
- moved R14 191.6 mm to (240.3, -27.5), turned to 90 degrees
- moved R15 191.6 mm to (237.8, -27.5), turned to 90 degrees
- moved R16 191.6 mm to (235.3, -27.5), turned to 90 degrees
- moved R17 191.6 mm to (232.8, -27.5), turned to 90 degrees
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Connections:
- J2 pad 1: (no net) -> PVDD
- J2 pad 10: (no net) -> COM2
- J2 pad 2: (no net) -> PVDD
- J2 pad 3: (no net) -> GND
- J2 pad 4: (no net) -> 2MOT_A
- J2 pad 5: (no net) -> GND
- J2 pad 6: (no net) -> 2MOT_B
- J2 pad 7: (no net) -> GND
- J2 pad 8: (no net) -> 2MOT_C
- J2 pad 9: (no net) -> GND
- J2 pad S1: (no net) -> GND
- J2 pad S2: (no net) -> GND
- J3 pad 1: (no net) -> PVDD
- J3 pad 10: (no net) -> COM3
- J3 pad 2: (no net) -> PVDD
- J3 pad 3: (no net) -> GND
- J3 pad 4: (no net) -> 3MOT_A
- J3 pad 5: (no net) -> GND
- J3 pad 6: (no net) -> 3MOT_B
- J3 pad 7: (no net) -> GND
- J3 pad 8: (no net) -> 3MOT_C
- J3 pad 9: (no net) -> GND
- J3 pad S1: (no net) -> GND
- J3 pad S2: (no net) -> GND
- J4 pad 1: (no net) -> PVDD
- J4 pad 10: (no net) -> COM4
- J4 pad 2: (no net) -> PVDD
- J4 pad 3: (no net) -> GND
- J4 pad 4: (no net) -> 4MOT_A
- J4 pad 5: (no net) -> GND
- J4 pad 6: (no net) -> 4MOT_B
- J4 pad 7: (no net) -> GND
- J4 pad 8: (no net) -> 4MOT_C
- J4 pad 9: (no net) -> GND
- J4 pad S1: (no net) -> GND
- J4 pad S2: (no net) -> GND
- J5 pad 1: (no net) -> PVDD
- J5 pad 10: (no net) -> COM5
- J5 pad 2: (no net) -> PVDD
- J5 pad 4: (no net) -> 5MOT_A
- J5 pad 6: (no net) -> 5MOT_B
- J5 pad 8: (no net) -> 5MOT_C
- J6 pad 1: (no net) -> PVDD
- J6 pad 10: (no net) -> COM6
- J6 pad 2: (no net) -> PVDD
- J6 pad 3: (no net) -> GND
- J6 pad 4: (no net) -> 6MOT_A
- J6 pad 5: (no net) -> GND
- J6 pad 6: (no net) -> 6MOT_B
- J6 pad 7: (no net) -> GND
- J6 pad 8: (no net) -> 6MOT_C
- J6 pad 9: (no net) -> GND
- J6 pad S1: (no net) -> GND
- J6 pad S2: (no net) -> GND
- J7 pad 1: (no net) -> PVDD
- J7 pad 10: (no net) -> COM7
- J7 pad 2: (no net) -> PVDD
- J7 pad 3: (no net) -> GND
- J7 pad 4: (no net) -> 7MOT_A
- J7 pad 5: (no net) -> GND
- J7 pad 6: (no net) -> 7MOT_B
- J7 pad 7: (no net) -> GND
- J7 pad 8: (no net) -> 7MOT_C
- J7 pad 9: (no net) -> GND
- J7 pad S1: (no net) -> GND
- J7 pad S2: (no net) -> GND
- J8 pad 1: (no net) -> PVDD
- J8 pad 10: (no net) -> COM8
- J8 pad 2: (no net) -> PVDD
- J8 pad 3: (no net) -> GND
- J8 pad 4: (no net) -> 8MOT_A
- J8 pad 5: (no net) -> GND
- J8 pad 6: (no net) -> 8MOT_B
- J8 pad 7: (no net) -> GND
- J8 pad 8: (no net) -> 8MOT_C
- J8 pad 9: (no net) -> GND
- J8 pad S1: (no net) -> GND
- J8 pad S2: (no net) -> GND
- JP4 pad 1: 5.0_VDC -> 5.0V
- U1 pad 10: COM_5 -> Net-(U1-PWM4)
- U1 pad 11: COM_6 -> Net-(U1-PWM5)
- U1 pad 12: COM_7 -> Net-(U1-PWM6)
- U1 pad 13: COM_8 -> Net-(U1-PWM7)
- U1 pad 15: (no net) -> unconnected-(U1-PWM8-Pad15)
- U1 pad 16: (no net) -> unconnected-(U1-PWM9-Pad16)
- U1 pad 17: (no net) -> unconnected-(U1-PWM10-Pad17)
- U1 pad 18: (no net) -> unconnected-(U1-PWM11-Pad18)
- U1 pad 19: (no net) -> unconnected-(U1-PWM12-Pad19)
- U1 pad 20: (no net) -> unconnected-(U1-PWM13-Pad20)
- U1 pad 21: (no net) -> unconnected-(U1-PWM14-Pad21)
- U1 pad 22: (no net) -> unconnected-(U1-PWM15-Pad22)
- U1 pad 6: COM_1 -> Net-(U1-PWM0)
- U1 pad 7: COM_2 -> Net-(U1-PWM1)
- U1 pad 8: COM_3 -> Net-(U1-PWM2)
- U1 pad 9: COM_4 -> Net-(U1-PWM3)
Routing:
- net COM_8: track 0.00 -> 29.1 mm
- net COM_7: track 0.00 -> 27.1 mm
- net COM_6: track 0.00 -> 24.6 mm
- net COM_5: track 0.12 -> 21.9 mm
- net COM_4: track 0.00 -> 19.2 mm
- net COM_3: track 0.14 -> 16.4 mm
- net COM_2: track 0.00 -> 13.6 mm
- net COM_1: track 0.00 -> 11.5 mm
- net SDA: track 12.8 -> 2.00 mm
- net SCL: track 13.0 -> 2.40 mm
- net OE: track 20.4 -> 12.6 mm
- net PVDD: vias 0 -> 25
- added copper zone on F.Cu, net PVDD
Other:
- board size 235 x 285 mm -> 285 x 235 mm

Commit message: Added connectors and esc footprints
Parts:
- removed the H1 at (90.8, -16.2)
- removed the H1 at (90.8, 33.8)
- removed the H1 at (307.2, 22.7)
- removed the H1 at (90.8, 83.8)
- removed the H1 at (231.2, 22.2)
- removed the H1 at (307.7, 122.2)
- removed the H1 at (232.2, 73.1)
- removed the H1 at (231.7, 122.6)
- removed J2, J3, J4, J5, J6, J7, J8: 10159560-A00221RLF, PowerDistroFootprints:AMPHENOL_10159560-A00221RLF
- added H1: M2.5, MountingHole:MountingHole_2.7mm_M2.5_ISO7380, F.Cu at (61.3, 128.0)
- added H2: M2.5, MountingHole:MountingHole_2.7mm_M2.5_ISO7380, F.Cu at (125.9, 128.0)
- added H3: M2.5, MountingHole:MountingHole_2.7mm_M2.5_ISO7380, F.Cu at (125.9, 166.0)
- added H4: M2.5, MountingHole:MountingHole_2.7mm_M2.5_ISO7380, F.Cu at (61.3, 166.0)
- moved J1 135.6 mm to (120.3, 147.0), turned to -90 degrees
- moved C1 96.4 mm to (213.4, 58.4)
- moved J9 96.4 mm to (173.3, 60.6)
- moved JP4 96.4 mm to (208.7, 53.7)
- moved LED1 96.4 mm to (203.7, 58.0)
- moved R1 96.4 mm to (256.2, 49.9)
- moved R10 96.4 mm to (204.5, 61.2)
- moved R11 96.4 mm to (221.9, 65.4)
- moved R12 96.4 mm to (219.4, 65.4)
- moved R13 96.4 mm to (216.9, 65.4)
- moved R14 96.4 mm to (214.4, 65.4)
- moved R15 96.4 mm to (211.9, 65.4)
- moved R16 96.4 mm to (209.4, 65.4)
- moved R17 96.4 mm to (206.9, 65.4)
- moved R18 96.4 mm to (204.4, 65.4)
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Routing:
- net 1MOT_C: track 0.00 -> 8.50 mm
- net 1MOT_B: track 0.00 -> 8.50 mm
- net 1MOT_A: track 0.00 -> 8.50 mm
- net GND: track 0.55 -> 0.79 mm, vias 0 -> 67
- net PVDD: vias 25 -> 30
- added copper zone on F.Cu, net 1MOT_A
- added copper zone on F.Cu, net 1MOT_B
- added copper zone on F.Cu, net 1MOT_C
- added copper zone on F.Cu, net GND
Other:
- board size 285 x 235 mm -> 275 x 225 mm

Commit message: changed motor controler numbers and hole numbers in PCB
Parts:
- added H10: M2.5, MountingHole:MountingHole_2.7mm_M2.5_ISO7380, F.Cu at (275.6, 128.2)
- added H11: M2.5, MountingHole:MountingHole_2.7mm_M2.5_ISO7380, F.Cu at (275.6, 166.1)
- added H12: M2.5, MountingHole:MountingHole_2.7mm_M2.5_ISO7380, F.Cu at (210.9, 166.1)
- added H13: M2.5, MountingHole:MountingHole_2.7mm_M2.5_ISO7380, F.Cu at (136.4, 175.2)
- added H14: M2.5, MountingHole:MountingHole_2.7mm_M2.5_ISO7380, F.Cu at (201.1, 175.2)
- added H15: M2.5, MountingHole:MountingHole_2.7mm_M2.5_ISO7380, F.Cu at (201.1, 213.1)
- added H16: M2.5, MountingHole:MountingHole_2.7mm_M2.5_ISO7380, F.Cu at (136.4, 213.1)
- added H17: M2.5, MountingHole:MountingHole_2.7mm_M2.5_ISO7380, F.Cu at (210.9, 175.2)
- added H18: M2.5, MountingHole:MountingHole_2.7mm_M2.5_ISO7380, F.Cu at (275.6, 175.2)
- added H19: M2.5, MountingHole:MountingHole_2.7mm_M2.5_ISO7380, F.Cu at (275.6, 213.1)
- added H20: M2.5, MountingHole:MountingHole_2.7mm_M2.5_ISO7380, F.Cu at (210.9, 213.1)
- added H21: M2.5, MountingHole:MountingHole_2.7mm_M2.5_ISO7380, F.Cu at (60.4, 222.2)
- added H22: M2.5, MountingHole:MountingHole_2.7mm_M2.5_ISO7380, F.Cu at (125.1, 222.2)
- added H23: M2.5, MountingHole:MountingHole_2.7mm_M2.5_ISO7380, F.Cu at (125.1, 260.1)
- added H24: M2.5, MountingHole:MountingHole_2.7mm_M2.5_ISO7380, F.Cu at (60.4, 260.1)
- added H25: M2.5, MountingHole:MountingHole_2.7mm_M2.5_ISO7380, F.Cu at (136.4, 222.2)
- added H26: M2.5, MountingHole:MountingHole_2.7mm_M2.5_ISO7380, F.Cu at (201.1, 222.2)
- added H27: M2.5, MountingHole:MountingHole_2.7mm_M2.5_ISO7380, F.Cu at (201.1, 260.1)
- added H28: M2.5, MountingHole:MountingHole_2.7mm_M2.5_ISO7380, F.Cu at (136.4, 260.1)
- added H29: M2.5, MountingHole:MountingHole_2.7mm_M2.5_ISO7380, F.Cu at (210.9, 222.2)
- added H30: M2.5, MountingHole:MountingHole_2.7mm_M2.5_ISO7380, F.Cu at (275.6, 222.2)
- added H31: M2.5, MountingHole:MountingHole_2.7mm_M2.5_ISO7380, F.Cu at (275.6, 260.1)
- added H32: M2.5, MountingHole:MountingHole_2.7mm_M2.5_ISO7380, F.Cu at (210.9, 260.1)
- added H5: M2.5, MountingHole:MountingHole_2.7mm_M2.5_ISO7380, F.Cu at (136.4, 128.2)
- added H6: M2.5, MountingHole:MountingHole_2.7mm_M2.5_ISO7380, F.Cu at (201.1, 128.2)
- added H7: M2.5, MountingHole:MountingHole_2.7mm_M2.5_ISO7380, F.Cu at (201.1, 166.1)
- added H8: M2.5, MountingHole:MountingHole_2.7mm_M2.5_ISO7380, F.Cu at (136.4, 166.1)
- added H9: M2.5, MountingHole:MountingHole_2.7mm_M2.5_ISO7380, F.Cu at (210.9, 128.2)
- added J2: 10159560-A00221RLF, PowerDistroFootprints:AMPHENOL_10159560-A00221RLF, F.Cu at (195.5, 147.2)
- added J3: 10159560-A00221RLF, PowerDistroFootprints:AMPHENOL_10159560-A00221RLF, F.Cu at (270.0, 147.2)
- added J4: 10159560-A00221RLF, PowerDistroFootprints:AMPHENOL_10159560-A00221RLF, F.Cu at (195.5, 194.2)
- added J5: 10159560-A00221RLF, PowerDistroFootprints:AMPHENOL_10159560-A00221RLF, F.Cu at (270.0, 194.2)
- added J6: 10159560-A00221RLF, PowerDistroFootprints:AMPHENOL_10159560-A00221RLF, F.Cu at (119.5, 241.2)
- added J7: 10159560-A00221RLF, PowerDistroFootprints:AMPHENOL_10159560-A00221RLF, F.Cu at (195.5, 241.2)
- added J8: 10159560-A00221RLF, PowerDistroFootprints:AMPHENOL_10159560-A00221RLF, F.Cu at (270.0, 241.2)
Routing:
- net 1MOT_C: track 8.50 -> 68.0 mm
- net 1MOT_B: track 8.50 -> 68.0 mm
- net 1MOT_A: track 8.50 -> 68.0 mm
- net GND: track 0.79 -> 2.48 mm, vias 67 -> 536
- net PVDD: vias 30 -> 240
Other:
- board size 275 x 225 mm -> 275 x 245 mm

Commit message: rearranged the power distro board
Parts:
- removed H25, H26, H27, H28: M2.5, MountingHole:MountingHole_2.7mm_M2.5_ISO7380
- added H29: MountingHole, MountingHole:MountingHole_2.7mm_M2.5_ISO7380, F.Cu at (214.0, 110.5)
- added H30: MountingHole, MountingHole:MountingHole_2.7mm_M2.5_ISO7380, F.Cu at (149.4, 110.5)
- added H31: MountingHole, MountingHole:MountingHole_2.7mm_M2.5_ISO7380, F.Cu at (149.4, 72.5)
- added H32: MountingHole, MountingHole:MountingHole_2.7mm_M2.5_ISO7380, F.Cu at (214.0, 72.5)
- added J10: ~, PowerDistroFootprints:MR30PW-M, F.Cu at (84.0, 42.5)
- added J11: ~, PowerDistroFootprints:MR30PW-M, F.Cu at (47.5, 232.5)
- added J12: ~, PowerDistroFootprints:MR30PW-M, F.Cu at (47.2, 210.2)
- added J13: ~, PowerDistroFootprints:MR30PW-M, F.Cu at (219.5, 41.5)
- added J14: ~, PowerDistroFootprints:MR30PW-M, F.Cu at (104.5, 42.5)
- added J15: ~, PowerDistroFootprints:MR30PW-M, F.Cu at (197.0, 41.5)
- added J16: ~, PowerDistroFootprints:MR30PW-M, F.Cu at (49.0, 123.0)
- added J17: ~, PowerDistroFootprints:MR30PW-M, F.Cu at (124.0, 43.0)
- H1, H10, H11, H12, H13, H14, H15, H16, H17, H18, H19, H2, H20, H21, H22, H23, H24, H29, H3, H30, H31, H32, H4, H5, H6, H7, H8, H9: value M2.5 -> MountingHole
- moved R1 297.1 mm to (-38.7, 13.5), turned to 180 degrees
- moved H24 296.5 mm to (290.0, 72.5), turned to 180 degrees
- moved TP1 293.3 mm to (-34.3, 13.5), turned to 0 degrees
- moved R2 291.5 mm to (-38.7, 18.5), turned to 180 degrees
- moved SW_A5 290.3 mm to (-30.7, 13.5), turned to 180 degrees
- moved TP2 287.7 mm to (-34.3, 18.5), turned to 0 degrees
- moved R3 286.1 mm to (-38.7, 23.5), turned to 180 degrees
- moved SW_A4 284.6 mm to (-30.7, 18.5), turned to 180 degrees
- moved TP3 282.2 mm to (-34.3, 23.5), turned to 0 degrees
- moved R4 280.7 mm to (-38.7, 28.5), turned to 180 degrees
- moved SW_A3 279.0 mm to (-30.7, 23.5), turned to 180 degrees
- moved TP4 276.7 mm to (-34.3, 28.5), turned to 0 degrees
- moved H31 276.5 mm to (72.6, 72.4), turned to 180 degrees
- moved R5 275.3 mm to (-38.7, 33.5), turned to 180 degrees
- moved SW_A2 273.4 mm to (-30.7, 28.5), turned to 180 degrees
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Connections:
- net COM_7 renamed COM7
- J2 pad 10: COM1 -> COM2
- J2 pad 4: 1MOT_A -> 2MOT_A
- J2 pad 6: 1MOT_B -> 2MOT_B
- J2 pad 8: 1MOT_C -> 2MOT_C
- J3 pad 10: COM1 -> COM3
- J3 pad 4: 1MOT_A -> 3MOT_A
- J3 pad 6: 1MOT_B -> 3MOT_B
- J3 pad 8: 1MOT_C -> 3MOT_C
- J4 pad 10: COM1 -> COM4
- J4 pad 4: 1MOT_A -> 4MOT_A
- J4 pad 6: 1MOT_B -> 4MOT_B
- J4 pad 8: 1MOT_C -> 4MOT_C
- J5 pad 10: COM1 -> COM5
- J5 pad 4: 1MOT_A -> 5MOT_A
- J5 pad 6: 1MOT_B -> 5MOT_B
- J5 pad 8: 1MOT_C -> 5MOT_C
- J6 pad 10: COM1 -> COM6
- J6 pad 4: 1MOT_A -> 6MOT_A
- J6 pad 6: 1MOT_B -> 6MOT_B
- J6 pad 8: 1MOT_C -> 6MOT_C
- J7 pad 10: COM1 -> COM8
- J7 pad 4: 1MOT_A -> 8MOT_A
- J7 pad 6: 1MOT_B -> 8MOT_B
- J7 pad 8: 1MOT_C -> 8MOT_C
- J8 pad 10: COM1 -> COM8
- J8 pad 4: 1MOT_A -> 8MOT_A
- J8 pad 6: 1MOT_B -> 8MOT_B
- J8 pad 8: 1MOT_C -> 8MOT_C
- R11 pad 2: COM_1 -> COM1
- R12 pad 2: COM_2 -> COM2
- R13 pad 2: COM_3 -> COM3
- R14 pad 2: COM_4 -> COM4
- R15 pad 2: COM_5 -> COM5
- R16 pad 2: COM_6 -> COM6
- R18 pad 2: COM_8 -> COM8
Routing:
- net Net-(U1-PWM7): track 0.00 -> 29.1 mm
- net COM_8: track 29.1 -> 0.00 mm
- net Net-(U1-PWM6): track 0.00 -> 27.1 mm
- net COM7: track 27.1 -> 0.00 mm
- net Net-(U1-PWM5): track 0.00 -> 24.6 mm
- net COM_6: track 24.6 -> 0.00 mm
- net Net-(U1-PWM4): track 0.12 -> 22.1 mm
- net COM_5: track 21.9 -> 0.00 mm
- net Net-(U1-PWM3): track 0.00 -> 19.2 mm
- net COM_4: track 19.2 -> 0.00 mm
- net COM_3: track 16.4 -> 0.00 mm
- net Net-(U1-PWM2): track 0.14 -> 16.6 mm
- net Net-(U1-PWM1): track 0.00 -> 13.6 mm
- net COM_2: track 13.6 -> 0.00 mm
- net (no net): track 0.00 -> 11.5 mm
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Other:
- board size 275 x 245 mm -> 280 x 230 mm
