File: 2024/PowerDistro/PowerDistro.kicad_pcb (KiCad board)
At the start: 4 copper layers, 280 x 230 mm, 83 parts, among them J1 10159560-A00221RLF, J2 10159560-A00221RLF, J3 10159560-A00221RLF, J4 10159560-A00221RLF, J5 10159560-A00221RLF, J6 10159560-A00221RLF, J7 10159560-A00221RLF, J8 10159560-A00221RLF, U1 PCA9685

Commit message: layed out the first set of traces for motor drivers
Parts:
- moved J10 323.5 mm to (367.5, 179.5), turned to -90 degrees
- moved J13 191.2 mm to (368.0, 162.0), turned to -90 degrees
- moved H14 127.2 mm to (350.0, 143.7), turned to -90 degrees
- moved H13 107.2 mm to (350.0, 79.0), turned to -90 degrees
- moved J11 104.6 mm to (138.0, 180.0)
- moved J4 101.8 mm to (332.2, 137.6), turned to 180 degrees
- moved LED1 100.4 mm to (68.9, 79.7)
- moved R11 100.4 mm to (76.3, 61.5)
- moved R12 100.4 mm to (76.3, 64.0)
- moved R13 100.4 mm to (76.3, 66.5)
- moved R14 100.4 mm to (76.3, 69.0)
- moved R15 100.4 mm to (76.3, 71.5)
- moved R16 100.4 mm to (76.3, 74.0)
- moved R17 100.4 mm to (76.3, 76.5)
- moved R18 100.4 mm to (76.3, 79.0)
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- renumbered J16 to J10, J10 to J17
Connections:
- J10 pad 1: 7MOT_A -> 1MOT_A
- J10 pad 2: 7MOT_B -> 1MOT_B
- J10 pad 3: 7MOT_C -> 1MOT_C
- J17 pad 1: 1MOT_A -> 8MOT_A
- J17 pad 2: 1MOT_B -> 8MOT_B
- J17 pad 3: 1MOT_C -> 8MOT_C
Routing:
- net 1MOT_B: track 68.0 -> 570.4 mm
- net 5MOT_C: track 0.00 -> 232.5 mm
- net 1MOT_C: track 67.9 -> 295.3 mm
- net 5MOT_A: track 0.00 -> 141.1 mm
- net 3MOT_A: track 8.50 -> 102.1 mm
- net 8MOT_A: track 0.00 -> 62.8 mm
- net 8MOT_B: track 0.00 -> 46.2 mm
- net 8MOT_C: track 0.00 -> 28.3 mm
- net 6MOT_C: track 0.00 -> 9.01 mm
- net 1MOT_A: track 59.5 -> 66.7 mm

Commit message: Pushing so Power connector can be added
Parts:
- removed H10, H11, H12, H13, H14, H15, H16, H17, H18, H19, H20, H21, H22, H23, H24, H29 (x2), H30 (x2), H31 (x2), H32 (x2), H5, H6, H7, H8, H9: MountingHole, MountingHole:MountingHole_2.7mm_M2.5_ISO7380
- removed the J10 at (367.5, 179.5)
- removed J11, J12, J13, J14, J15, J17 (x2): ~, PowerDistroFootprints:MR30PW-M
- removed J2, J3, J4, J5, J6, J7, J8: 10159560-A00221RLF, PowerDistroFootprints:AMPHENOL_10159560-A00221RLF
- added H1: MountingHole, MountingHole:MountingHole_2.7mm_M2.5_ISO7380, F.Cu at (234.6, 158.9)
- added H1: MountingHole, MountingHole:MountingHole_2.7mm_M2.5_ISO7380, F.Cu at (282.1, 158.9)
- added H1: MountingHole, MountingHole:MountingHole_2.7mm_M2.5_ISO7380, F.Cu at (291.4, 109.6)
- added H1: MountingHole, MountingHole:MountingHole_2.7mm_M2.5_ISO7380, F.Cu at (339.0, 109.5)
- added H1: MountingHole, MountingHole:MountingHole_2.7mm_M2.5_ISO7380, F.Cu at (195.4, 109.6)
- added H1: MountingHole, MountingHole:MountingHole_2.7mm_M2.5_ISO7380, F.Cu at (242.9, 110.1)
- added H1: MountingHole, MountingHole:MountingHole_2.7mm_M2.5_ISO7380, F.Cu at (329.1, 159.9)
- added H2: MountingHole, MountingHole:MountingHole_2.7mm_M2.5_ISO7380, F.Cu at (291.4, 44.9)
- added H2: MountingHole, MountingHole:MountingHole_2.7mm_M2.5_ISO7380, F.Cu at (339.0, 44.9)
- added H2: MountingHole, MountingHole:MountingHole_2.7mm_M2.5_ISO7380, F.Cu at (195.4, 44.9)
- added H2: MountingHole, MountingHole:MountingHole_2.7mm_M2.5_ISO7380, F.Cu at (234.6, 223.6)
- added H2: MountingHole, MountingHole:MountingHole_2.7mm_M2.5_ISO7380, F.Cu at (282.1, 223.6)
- added H2: MountingHole, MountingHole:MountingHole_2.7mm_M2.5_ISO7380, F.Cu at (329.1, 224.6)
- added H2: MountingHole, MountingHole:MountingHole_2.7mm_M2.5_ISO7380, F.Cu at (242.9, 45.4)
- added H3: MountingHole, MountingHole:MountingHole_2.7mm_M2.5_ISO7380, F.Cu at (233.4, 44.9)
- added H3: MountingHole, MountingHole:MountingHole_2.7mm_M2.5_ISO7380, F.Cu at (329.4, 44.9)
- added H3: MountingHole, MountingHole:MountingHole_2.7mm_M2.5_ISO7380, F.Cu at (377.0, 44.9)
- added H3: MountingHole, MountingHole:MountingHole_2.7mm_M2.5_ISO7380, F.Cu at (291.1, 224.6)
- added H3: MountingHole, MountingHole:MountingHole_2.7mm_M2.5_ISO7380, F.Cu at (280.9, 45.4)
- added H3: MountingHole, MountingHole:MountingHole_2.7mm_M2.5_ISO7380, F.Cu at (196.6, 223.6)
- added H3: MountingHole, MountingHole:MountingHole_2.7mm_M2.5_ISO7380, F.Cu at (244.1, 223.6)
- added H4: MountingHole, MountingHole:MountingHole_2.7mm_M2.5_ISO7380, F.Cu at (233.4, 109.6)
- added H4: MountingHole, MountingHole:MountingHole_2.7mm_M2.5_ISO7380, F.Cu at (244.1, 158.9)
- added H4: MountingHole, MountingHole:MountingHole_2.7mm_M2.5_ISO7380, F.Cu at (329.4, 109.6)
- added H4: MountingHole, MountingHole:MountingHole_2.7mm_M2.5_ISO7380, F.Cu at (196.6, 158.9)
- added H4: MountingHole, MountingHole:MountingHole_2.7mm_M2.5_ISO7380, F.Cu at (291.1, 159.9)
- added H4: MountingHole, MountingHole:MountingHole_2.7mm_M2.5_ISO7380, F.Cu at (280.9, 110.1)
- added H4: MountingHole, MountingHole:MountingHole_2.7mm_M2.5_ISO7380, F.Cu at (377.0, 109.5)
- added J1: 10159560-A00221RLF, PowerDistroFootprints:AMPHENOL_10159560-A00221RLF, F.Cu at (260.9, 51.5)
- added J1: 10159560-A00221RLF, PowerDistroFootprints:AMPHENOL_10159560-A00221RLF, F.Cu at (357.0, 50.9)
- added J1: 10159560-A00221RLF, PowerDistroFootprints:AMPHENOL_10159560-A00221RLF, F.Cu at (311.1, 218.5)
- added J1: 10159560-A00221RLF, PowerDistroFootprints:AMPHENOL_10159560-A00221RLF, F.Cu at (213.4, 51.0)
- added J1: 10159560-A00221RLF, PowerDistroFootprints:AMPHENOL_10159560-A00221RLF, F.Cu at (309.4, 51.0)
- added J1: 10159560-A00221RLF, PowerDistroFootprints:AMPHENOL_10159560-A00221RLF, F.Cu at (216.6, 217.5)
- added J1: 10159560-A00221RLF, PowerDistroFootprints:AMPHENOL_10159560-A00221RLF, F.Cu at (264.1, 217.5)
- added J10: ~, PowerDistroFootprints:MR30PB, F.Cu at (266.6, 234.4)
- added J10: ~, PowerDistroFootprints:MR30PB, F.Cu at (219.1, 234.4)
- added J10: ~, PowerDistroFootprints:MR30PB, F.Cu at (313.6, 235.4)
- added J10: ~, PowerDistroFootprints:MR30PB, F.Cu at (258.4, 34.6)
- added J10: ~, PowerDistroFootprints:MR30PB, F.Cu at (354.5, 34.0)
- added J10: ~, PowerDistroFootprints:MR30PB, F.Cu at (210.9, 34.1)
- added J10: ~, PowerDistroFootprints:MR30PB, F.Cu at (361.5, 235.5)
- added J10: ~, PowerDistroFootprints:MR30PB, F.Cu at (306.9, 34.1)
- moved J9 284.6 mm to (355.2, 133.0), turned to 90 degrees
- moved H1 73.5 mm to (377.0, 160.0), turned to -90 degrees
- moved H2 64.1 mm to (377.0, 224.7), turned to -90 degrees
- moved H4 52.8 mm to (339.0, 160.0), turned to -90 degrees
- moved J1 39.5 mm to (359.0, 218.6), turned to 180 degrees
- moved H3 38.8 mm to (339.0, 224.7), turned to -90 degrees
- moved JP4 9.15 mm to (55.5, 74.3)
Routing:
- net 1MOT_B: track 570.4 -> 0.00 mm
- net 1MOT_C: track 295.3 -> 0.00 mm
- net 5MOT_C: track 232.5 -> 0.00 mm
- net 5MOT_A: track 141.1 -> 0.00 mm
- net 3MOT_A: track 102.1 -> 0.00 mm
- net 1MOT_A: track 66.7 -> 0.00 mm
- net 8MOT_A: track 62.8 -> 0.00 mm
- net 8MOT_B: track 46.2 -> 0.00 mm
- net 8MOT_C: track 28.3 -> 0.00 mm
- net 6MOT_C: track 9.01 -> 0.00 mm

Commit message: renamed the motor controllers
Parts:
- moved JP4 264.5 mm to (316.0, 120.0), turned to 0 degrees
- moved R7 227.7 mm to (272.3, 139.7), turned to 180 degrees
- moved LED1 226.0 mm to (289.5, 128.9), turned to -90 degrees
- moved R9 224.8 mm to (279.9, 133.5), turned to 0 degrees
- moved R8 221.7 mm to (279.9, 131.0), turned to 180 degrees
- moved R10 221.5 mm to (288.7, 125.7), turned to 180 degrees
- moved U1 220.0 mm to (272.4, 133.6), turned to -90 degrees
- moved C1 218.5 mm to (279.8, 128.5), turned to 0 degrees
- moved R6 218.3 mm to (262.0, 137.0), turned to -90 degrees
- moved R18 216.7 mm to (288.8, 121.5), turned to -90 degrees
- moved R5 215.8 mm to (257.0, 137.0), turned to -90 degrees
- moved R17 214.8 mm to (286.3, 121.5), turned to -90 degrees
- moved R4 213.4 mm to (252.0, 137.0), turned to -90 degrees
- moved R16 212.9 mm to (283.8, 121.5), turned to -90 degrees
- moved TP6 212.7 mm to (262.0, 132.7), turned to 90 degrees
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- renumbered H2 to H10, H3 to H11, H4 to H12, H1 to H13, H2 to H14, H3 to H15, H4 to H16, H1 to H17, H2 to H18, H3 to H19, H4 to H20, H1 to H21, H2 to H22, H3 to H23, H4 to H24, H1 to H25, H2 to H26, H3 to H27, H4 to H28, H1 to H29, H2 to H30, H3 to H31, H4 to H32, H1 to H5, H2 to H6, H3 to H7, H4 to H8, H1 to H9, J10 to J11, J10 to J12, J10 to J13, J10 to J14, J10 to J15, J10 to J16, J10 to J17, J1 to J2, J1 to J3, J1 to J4, J1 to J5, J1 to J6, J1 to J7, J1 to J8
Connections:
- J11 pad 1: 1MOT_A -> 2MOT_A
- J11 pad 2: 1MOT_B -> 2MOT_B
- J11 pad 3: 1MOT_C -> 2MOT_C
- J12 pad 1: 1MOT_A -> 3MOT_A
- J12 pad 2: 1MOT_B -> 3MOT_B
- J12 pad 3: 1MOT_C -> 3MOT_C
- J13 pad 1: 1MOT_A -> 4MOT_A
- J13 pad 2: 1MOT_B -> 4MOT_B
- J13 pad 3: 1MOT_C -> 4MOT_C
- J14 pad 1: 1MOT_A -> 5MOT_A
- J14 pad 2: 1MOT_B -> 5MOT_B
- J14 pad 3: 1MOT_C -> 5MOT_C
- J15 pad 1: 1MOT_A -> 6MOT_A
- J15 pad 2: 1MOT_B -> 6MOT_B
- J15 pad 3: 1MOT_C -> 6MOT_C
- J16 pad 1: 1MOT_A -> 7MOT_A
- J16 pad 2: 1MOT_B -> 7MOT_B
- J16 pad 3: 1MOT_C -> 7MOT_C
- J17 pad 1: 1MOT_A -> 8MOT_A
- J17 pad 2: 1MOT_B -> 8MOT_B
- J17 pad 3: 1MOT_C -> 8MOT_C
- J2 pad 10: COM1 -> COM2
- J2 pad 4: 1MOT_A -> 2MOT_A
- J2 pad 6: 1MOT_B -> 2MOT_B
- J2 pad 8: 1MOT_C -> 2MOT_C
- J3 pad 10: COM1 -> COM3
- J3 pad 4: 1MOT_A -> 3MOT_A
- J3 pad 6: 1MOT_B -> 3MOT_B
- J3 pad 8: 1MOT_C -> 3MOT_C
- J4 pad 10: COM1 -> COM4
- J4 pad 4: 1MOT_A -> 4MOT_A
- J4 pad 6: 1MOT_B -> 4MOT_B
- J4 pad 8: 1MOT_C -> 4MOT_C
- J5 pad 10: COM1 -> COM5
- J5 pad 4: 1MOT_A -> 5MOT_A
- J5 pad 6: 1MOT_B -> 5MOT_B
- J5 pad 8: 1MOT_C -> 5MOT_C
- J6 pad 10: COM1 -> COM6
- J6 pad 4: 1MOT_A -> 6MOT_A
- J6 pad 6: 1MOT_B -> 6MOT_B
- J6 pad 8: 1MOT_C -> 6MOT_C
- J7 pad 10: COM1 -> COM7
- J7 pad 4: 1MOT_A -> 7MOT_A
- J7 pad 6: 1MOT_B -> 7MOT_B
- J7 pad 8: 1MOT_C -> 7MOT_C
- J8 pad 10: COM1 -> COM8
- J8 pad 4: 1MOT_A -> 8MOT_A
- J8 pad 6: 1MOT_B -> 8MOT_B
- J8 pad 8: 1MOT_C -> 8MOT_C
Routing:
- net OE: track 12.6 -> 8.34 mm
- net SCL: track 2.40 -> 0.00 mm
- net SDA: track 2.00 -> 0.00 mm
- net GND: track 2.48 -> 1.93 mm
- added copper zone on F.Cu, net 2MOT_A
- added copper zone on F.Cu, net 2MOT_B
- added copper zone on F.Cu, net 2MOT_C
- added copper zone on F.Cu, net 3MOT_A
- added copper zone on F.Cu, net 3MOT_B
- added copper zone on F.Cu, net 3MOT_C
- added copper zone on F.Cu, net 4MOT_A
- added copper zone on F.Cu, net 4MOT_B
- added copper zone on F.Cu, net 4MOT_C
- added copper zone on F.Cu, net 5MOT_A
- added copper zone on F.Cu, net 5MOT_B
- added copper zone on F.Cu, net 5MOT_C
- added copper zone on F.Cu, net 6MOT_A
- added copper zone on F.Cu, net 6MOT_B
- added copper zone on F.Cu, net 6MOT_C
- added copper zone on F.Cu, net 7MOT_A
- added copper zone on F.Cu, net 7MOT_B
- added copper zone on F.Cu, net 7MOT_C
- added copper zone on F.Cu, net 8MOT_A
- added copper zone on F.Cu, net 8MOT_B
- added copper zone on F.Cu, net 8MOT_C

Commit message: Added Vertical Connector Footprints, Fixed MR-30 symbol
Parts:
- removed JP4: SM06B-GHS-TB_LF__SN_, PowerDistroFootprints:JST_SM06B-GHS-TB_LF__SN_
- moved H20 1.93 mm to (232.4, 107.9)
- moved J5 1.93 mm to (212.4, 49.4)
- moved J14 1.93 mm to (209.9, 32.5)
- moved H19 1.93 mm to (232.4, 43.3)
- moved H17 1.93 mm to (194.4, 107.9)
- moved H18 1.93 mm to (194.4, 43.3)
- moved J2 1.42 mm to (312.2, 217.6)
- moved H1 1.42 mm to (378.1, 159.2)
- moved H2 1.42 mm to (378.1, 223.8)
- moved H3 1.42 mm to (340.1, 223.8)
- moved H4 1.42 mm to (340.1, 159.2)
- moved J11 1.42 mm to (314.7, 234.5)
- moved H5 1.42 mm to (330.2, 159.1)
- moved H6 1.42 mm to (330.2, 223.7)
- moved H7 1.42 mm to (292.3, 223.7)
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
Commit message: Added power layer to power distro motors
Parts:
- removed LED1: GREEN, LED_SMD:LED_0603_1608Metric
- removed R10: 470, Resistor_SMD:R_0603_1608Metric
- added H33: MountingHole, MountingHole:MountingHole_4.3mm_M4_ISO7380, F.Cu at (118.5, 24.5)
- added H34: MountingHole, MountingHole:MountingHole_4.3mm_M4_ISO7380, F.Cu at (387.0, 24.5)
- added H35: MountingHole, MountingHole:MountingHole_4.3mm_M4_ISO7380, F.Cu at (387.0, 241.5)
- added H36: MountingHole, MountingHole:MountingHole_4.3mm_M4_ISO7380, F.Cu at (118.5, 242.0)
- added J18: Conn_01x02_Pin, PowerDistroFootprints:XT90PB, F.Cu at (186.5, 134.8)
- added J19: 4 Pin JST-GH, PowerDistroFootprints:JST_BM04B-GHS-TBT_LF__SN__N_, F.Cu at (255.9, 119.5)
- added J20: 4 Pin JST-GH, PowerDistroFootprints:JST_BM04B-GHS-TBT_LF__SN__N_, F.Cu at (248.2, 119.5)
- added J21: 4 Pin JST-GH, PowerDistroFootprints:JST_BM04B-GHS-TBT_LF__SN__N_, F.Cu at (240.5, 119.5)
- added J22: 4 Pin JST-GH, PowerDistroFootprints:JST_BM04B-GHS-TBT_LF__SN__N_, F.Cu at (232.8, 119.5)
- moved R1 13.9 mm to (235.5, 150.8)
- moved R2 13.9 mm to (240.5, 150.8)
- moved R3 13.9 mm to (245.5, 150.8)
- moved R4 13.9 mm to (250.5, 150.8)
- moved R5 13.9 mm to (255.5, 150.8)
- moved R6 13.9 mm to (260.5, 150.8)
- moved SW_A0 13.9 mm to (260.5, 142.8)
- moved SW_A1 13.9 mm to (255.5, 142.8)
- moved SW_A2 13.9 mm to (250.5, 142.8)
- moved SW_A3 13.9 mm to (245.5, 142.8)
- moved SW_A4 13.9 mm to (240.5, 142.8)
- moved SW_A5 13.9 mm to (235.5, 142.8)
- moved TP1 13.9 mm to (235.5, 146.5)
- moved TP2 13.9 mm to (240.5, 146.5)
- moved TP3 13.9 mm to (245.5, 146.5)
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Connections:
- net OE renamed Net-(U1-#OE)
- R8 pad 2: SCL -> I2C2_CLK
- R9 pad 2: SDA -> I2C2_DAT
- U1 pad 26: SCL -> I2C2_CLK
- U1 pad 27: SDA -> I2C2_DAT
Routing:
- added copper zone on In1.Cu, net GND
- added copper zone on B.Cu, net PVDD
- removed copper zone on In1.Cu, net 5.0_VDC

Commit message: wired the PCA and Orin connecter together and added motor controller comms
Parts:
- moved J22 134.2 mm to (366.5, 130.7), turned to 90 degrees
- moved J21 118.9 mm to (358.9, 130.7), turned to 90 degrees
- moved J20 103.6 mm to (351.2, 130.7), turned to 90 degrees
- moved J19 88.4 mm to (343.5, 130.7), turned to 90 degrees
- moved R1 75.8 mm to (311.3, 151.0)
- moved R2 75.8 mm to (316.3, 151.0)
- moved R3 75.8 mm to (321.3, 151.0)
- moved R4 75.8 mm to (326.3, 151.0)
- moved R5 75.8 mm to (331.3, 151.0)
- moved R6 75.8 mm to (336.3, 151.0)
- moved SW_A0 75.8 mm to (336.3, 143.0)
- moved SW_A1 75.8 mm to (331.3, 143.0)
- moved SW_A2 75.8 mm to (326.3, 143.0)
- moved SW_A3 75.8 mm to (321.3, 143.0)
- moved SW_A4 75.8 mm to (316.3, 143.0)
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Connections:
- C1 pad 1: VCC -> 3.3_VDC
- J19 pad S1: (no net) -> GND
- J19 pad S2: (no net) -> GND
- J20 pad S1: (no net) -> GND
- J20 pad S2: (no net) -> GND
- J21 pad S1: (no net) -> GPIO17
- J21 pad S2: (no net) -> GND
- J22 pad S1: (no net) -> GND
- J22 pad S2: (no net) -> GND
- R8 pad 1: VCC -> 3.3_VDC
- R9 pad 1: VCC -> 3.3_VDC
- SW_A0 pad 1: VCC -> 3.3_VDC
- SW_A1 pad 1: VCC -> 3.3_VDC
- SW_A2 pad 1: VCC -> 3.3_VDC
- SW_A3 pad 1: VCC -> 3.3_VDC
- SW_A4 pad 1: VCC -> 3.3_VDC
- SW_A5 pad 1: VCC -> 3.3_VDC
- U1 pad 28: VCC -> 3.3_VDC
Routing:
- net COM4: track 0.00 -> 188.7 mm
- net COM5: track 0.00 -> 155.2 mm
- net COM3: track 0.00 -> 138.2 mm
- net COM8: track 0.00 -> 119.4 mm
- net COM1: track 0.00 -> 119.3 mm
- net COM6: track 0.00 -> 103.8 mm
- net COM2: track 0.00 -> 88.2 mm
- net COM7: track 0.00 -> 74.7 mm
- net I2C2_CLK: track 0.00 -> 65.7 mm
- net I2C2_DAT: track 0.00 -> 60.0 mm
- net 3.3_VDC: track 0.00 -> 53.8 mm, vias 0 -> 7
- net A5: track 3.00 -> 26.9 mm
- net A4: track 3.00 -> 18.7 mm
- net A0: track 3.00 -> 18.3 mm
- net A1: track 3.00 -> 18.1 mm
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- added copper zone on In2.Cu, net 3.3_VDC
- removed copper zone on In2.Cu, net GND
Other:
- outline, holes or cut-outs redrawn
