File: 2025/BatteryProtection/BatteryProtection.kicad_pcb (KiCad board)
At the start: 4 copper layers, 90.9 x 36.6 mm, 43 parts, among them J1 Screw_Terminal_01x02, J2 Screw_Terminal_01x02, Q1 FDMS8333L, Q2 FDMS8333L, Q3 FDMS8333L, Q4 FDMS8333L, U1 MAX25431ATGA/VY+

Commit message: Started on PCB
Parts:
- removed C10, C11, C6, C7, C8: 22u, Capacitor_SMD:C_1812_4532Metric
- removed C9: 120p, Capacitor_SMD:C_0603_1608Metric
- removed D3: DFLS160-7, Diode_SMD:D_SOD-123
- removed D4, D5, D6, D7: BAT54XV2T1G, Diode_SMD:D_SOD-523
- removed J1, J2: Screw_Terminal_01x02, TerminalBlock_Phoenix:TerminalBlock_Phoenix_MKDS-1,5-2_1x02_P5.00mm_Horizontal
- removed L1: 13uH, AllenControlsBuckBoost:L_Wuerth_HCI-1365
- removed TP1: VCC, TestPoint:TestPoint_Pad_1.5x1.5mm
- added Q10: BC849, Package_TO_SOT_SMD:SOT-23, F.Cu at (137.5, 109.5)
- added Q11: BC849, Package_TO_SOT_SMD:SOT-23, F.Cu at (132.6, 109.5)
- added Q5: BC849, Package_TO_SOT_SMD:SOT-23, F.Cu at (138.9, 104.1)
- added Q6: BC849, Package_TO_SOT_SMD:SOT-23, F.Cu at (134.2, 104.1)
- added Q7: BC849, Package_TO_SOT_SMD:SOT-23, F.Cu at (152.8, 109.0)
- added Q8: BC849, Package_TO_SOT_SMD:SOT-23, F.Cu at (148.1, 109.0)
- added Q9: BC849, Package_TO_SOT_SMD:SOT-23, F.Cu at (142.9, 109.5)
- added R17: 1k, Resistor_SMD:R_0603_1608Metric_Pad0.98x0.95mm_HandSolder, F.Cu at (112.9, 90.5)
- added R18: 1k, Resistor_SMD:R_0603_1608Metric_Pad0.98x0.95mm_HandSolder, F.Cu at (112.9, 88.0)
- added R19: 1k, Resistor_SMD:R_0603_1608Metric_Pad0.98x0.95mm_HandSolder, F.Cu at (112.9, 85.5)
- added R20: 1k, Resistor_SMD:R_0603_1608Metric_Pad0.98x0.95mm_HandSolder, F.Cu at (108.5, 103.0)
- added R21: 1k, Resistor_SMD:R_0603_1608Metric_Pad0.98x0.95mm_HandSolder, F.Cu at (108.5, 100.5)
- added R22: 1k, Resistor_SMD:R_0603_1608Metric_Pad0.98x0.95mm_HandSolder, F.Cu at (108.5, 98.0)
- added R23: 1k, Resistor_SMD:R_0603_1608Metric_Pad0.98x0.95mm_HandSolder, F.Cu at (108.5, 95.5)
- added U2: PLACEHOLDER, Package_TO_SOT_SMD:SOT-23-5, F.Cu at (139.4, 94.0)
- C1, C2: value 100n -> 10nF; footprint Capacitor_SMD:C_0603_1608Metric -> Capacitor_SMD:C_0603_1608Metric_Pad1.08x0.95mm_HandSolder
- C3: value 22u -> 1uF; footprint Capacitor_SMD:C_1812_4532Metric -> Capacitor_SMD:C_0603_1608Metric_Pad1.08x0.95mm_HandSolder
- C4: value 4.7u -> 1uF; footprint Capacitor_SMD:C_1210_3225Metric -> Capacitor_SMD:C_0603_1608Metric_Pad1.08x0.95mm_HandSolder
- C5: value 36n -> 0.1uF; footprint Capacitor_SMD:C_0603_1608Metric -> Capacitor_SMD:C_0603_1608Metric_Pad1.08x0.95mm_HandSolder
- D1: value LED -> 4.7V; footprint LED_SMD:LED_0805_2012Metric -> Diode_SMD:D_0603_1608Metric_Pad1.05x0.95mm_HandSolder
- D2: value DFLS160-7 -> 5.6V; footprint Diode_SMD:D_SOD-123 -> Diode_SMD:D_0603_1608Metric_Pad1.05x0.95mm_HandSolder
- Q1: value FDMS8333L -> IXTA140P05T; footprint Package_TO_SOT_SMD:TDSON-8-1 -> Package_TO_SOT_SMD:TO-263-2
- Q2, Q3, Q4: value FDMS8333L -> BC849; footprint Package_TO_SOT_SMD:TDSON-8-1 -> Package_TO_SOT_SMD:SOT-23
- R1: value 6m -> 100k; footprint Resistor_SMD:R_2010_5025Metric -> Resistor_SMD:R_0603_1608Metric_Pad0.98x0.95mm_HandSolder
- R10: value 182k -> 100k; footprint Resistor_SMD:R_0402_1005Metric -> Resistor_SMD:R_0603_1608Metric_Pad0.98x0.95mm_HandSolder
- R11: value 4.7 -> Load; footprint Resistor_SMD:R_0603_1608Metric -> Resistor_SMD:R_0603_1608Metric_Pad0.98x0.95mm_HandSolder
- R12: value 6.19k -> 100k; footprint Resistor_SMD:R_0402_1005Metric -> Resistor_SMD:R_0603_1608Metric_Pad0.98x0.95mm_HandSolder
- R13: value 10k -> 100k; footprint Resistor_SMD:R_0402_1005Metric -> Resistor_SMD:R_0603_1608Metric_Pad0.98x0.95mm_HandSolder
- R14: value 4.7 -> 100k; footprint Resistor_SMD:R_0603_1608Metric -> Resistor_SMD:R_0603_1608Metric_Pad0.98x0.95mm_HandSolder
- R15, R16: value 4.7 -> 1k; footprint Resistor_SMD:R_0603_1608Metric -> Resistor_SMD:R_0603_1608Metric_Pad0.98x0.95mm_HandSolder
- R2: value 6m -> 50k; footprint Resistor_SMD:R_2010_5025Metric -> Resistor_SMD:R_0603_1608Metric_Pad0.98x0.95mm_HandSolder
- R3: footprint Resistor_SMD:R_0402_1005Metric -> Resistor_SMD:R_0603_1608Metric_Pad0.98x0.95mm_HandSolder
- R4: value 2.2k -> 10k; footprint Resistor_SMD:R_0402_1005Metric -> Resistor_SMD:R_0603_1608Metric_Pad0.98x0.95mm_HandSolder
- R5, R7: value 1 -> 1k; footprint Resistor_SMD:R_0603_1608Metric -> Resistor_SMD:R_0603_1608Metric_Pad0.98x0.95mm_HandSolder
- R6: value 10k -> 1k; footprint Resistor_SMD:R_0402_1005Metric -> Resistor_SMD:R_0603_1608Metric_Pad0.98x0.95mm_HandSolder
- R8: value 41.2 -> 100k; footprint Resistor_SMD:R_0402_1005Metric -> Resistor_SMD:R_0603_1608Metric_Pad0.98x0.95mm_HandSolder
- R9: value 73.2k -> 1k; footprint Resistor_SMD:R_0402_1005Metric -> Resistor_SMD:R_0603_1608Metric_Pad0.98x0.95mm_HandSolder
- U1: value MAX25431ATGA/VY+ -> PLACEHOLDER; footprint AllenControlsBuckBoost:21-100290_MXM -> Package_TO_SOT_SMD:SOT-23-5
- moved Q1 48.0 mm to (171.9, 89.0), turned to 0 degrees
- moved R15 45.4 mm to (112.9, 95.5), turned to 180 degrees
- moved R16 44.7 mm to (112.9, 93.0), turned to 180 degrees
- moved R2 40.8 mm to (121.5, 94.4), turned to -90 degrees
- moved C5 30.6 mm to (157.1, 86.5)
- moved R7 30.1 mm to (117.2, 95.5), turned to 180 degrees
- moved R10 27.6 mm to (117.2, 88.0), turned to 180 degrees
- moved R3 27.5 mm to (125.5, 88.1), turned to -90 degrees
- moved R4 27.5 mm to (128.0, 88.1), turned to -90 degrees
- moved R9 26.6 mm to (117.2, 90.5), turned to 180 degrees
- moved R12 25.0 mm to (112.9, 103.0), turned to 180 degrees
- moved Q3 24.3 mm to (148.6, 90.0), turned to 0 degrees
- moved R13 21.6 mm to (112.9, 100.5), turned to 180 degrees
- moved R8 20.9 mm to (117.2, 93.0), turned to 180 degrees
- moved D1 20.1 mm to (132.0, 96.4), turned to -90 degrees
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Connections:
- C1 pad 2: /LX1 -> GND
- C2 pad 1: /LX2 -> Net-(D1-K)
- C2 pad 2: Net-(D3-K) -> GND
- C3 pad 1: VIN -> GND
- C3 pad 2: GND -> Vs
- C4 pad 1: VCC -> GND
- C4 pad 2: GND -> Vs
- C5 pad 1: Net-(U1-COMP) -> Net-(Q2-E)
- C5 pad 2: Net-(C5-Pad2) -> Net-(Q1-G)
- D1 pad 1: GND -> Net-(D1-K)
- D1 pad 2: Net-(D1-A) -> GND
- D2 pad 2: Net-(D2-A) -> GND
- Q1 pad 1: /LX1 -> Net-(Q1-G)
- Q1 pad 2: /LX1 -> Vs
- Q1 pad 3: /LX1 -> Net-(Q1-S)
- Q2 pad 1: /LX2 -> Net-(Q2-B)
- Q2 pad 2: /LX2 -> Net-(Q2-E)
- Q2 pad 3: /LX2 -> Vs
- Q3 pad 1: GND -> Net-(Q3-B)
- Q3 pad 2: GND -> Net-(Q2-E)
- Q3 pad 3: GND -> Vs
- Q4 pad 1: GND -> Net-(Q4-B)
- Q4 pad 2: GND -> Net-(Q2-E)
- Q4 pad 3: GND -> Vs
- R1 pad 1: VIN -> Vs
- R1 pad 2: /CSN1 -> Net-(U1-+)
- R10 pad 1: Net-(U1-FB) -> Net-(Q1-G)
- R10 pad 2: VOUT -> Vs
- R11 pad 1: /DH1 -> GND
- R11 pad 2: Net-(D4-K) -> Net-(Q1-S)
- R12 pad 1: GND -> Net-(Q5-C)
- R12 pad 2: Net-(C5-Pad2) -> Vs
- R13 pad 1: GND -> Net-(Q6-C)
- R13 pad 2: Net-(U1-FB) -> Vs
- R14 pad 1: /DL1 -> Net-(Q8-C)
- R14 pad 2: Net-(D5-K) -> Vs
- R15 pad 1: /DH2 -> Net-(Q6-C)
- R15 pad 2: Net-(D6-K) -> Net-(Q8-B)
- R16 pad 1: /DL2 -> Net-(Q9-C)
- R16 pad 2: Net-(D7-K) -> Net-(Q7-B)
- R2 pad 1: VOUT -> Net-(U1-+)
- R2 pad 2: /CSP2 -> GND
- R3 pad 1: /PGOOD -> Vs
- R3 pad 2: VCC -> Net-(D2-K)
- R4 pad 1: Net-(D1-A) -> Vs
- R4 pad 2: /PGOOD -> Net-(D1-K)
- R5 pad 1: Net-(D2-A) -> Net-(Q2-B)
- R5 pad 2: VCC -> Net-(R5-Pad2)
- R6 pad 1: VIN -> Net-(R6-Pad1)
- R6 pad 2: Net-(U1-EN) -> Net-(Q3-B)
- R7 pad 1: Net-(D3-A) -> Net-(Q8-C)
- R7 pad 2: VCC -> Net-(Q4-B)
- R8 pad 2: Net-(U1-SLP) -> Net-(Q2-E)
- R9 pad 1: GND -> Net-(Q1-G)
- R9 pad 2: Net-(U1-FSW) -> Net-(Q2-E)
- U1 pad 1: /DL1 -> Net-(D2-K)
- U1 pad 3: /CSN1 -> Net-(U1-+)
- U1 pad 4: VIN -> Net-(R5-Pad2)
- U1 pad 5: VIN -> Vs
Routing:
- net VOUT: track 98.6 -> 0.00 mm, vias 5 -> 0
- net VIN: track 87.9 -> 0.00 mm, vias 4 -> 0
- net VCC: track 57.4 -> 0.00 mm
- net /DH1: track 49.1 -> 0.00 mm, vias 2 -> 0
- net /CSN1: track 46.0 -> 0.00 mm, vias 2 -> 0
- net /CSP2: track 44.6 -> 0.00 mm, vias 2 -> 0
- net /DH2: track 34.7 -> 0.00 mm, vias 2 -> 0
- net /DL2: track 20.1 -> 0.00 mm
- net /LX1: track 18.0 -> 0.00 mm
- net /LX2: track 17.7 -> 0.00 mm
- net /DL1: track 15.0 -> 0.00 mm
- net GND: track 14.8 -> 0.00 mm, vias 153 -> 0
- net Net-(U1-FB): track 8.15 -> 0.00 mm
- net Net-(D2-K): track 6.16 -> 0.00 mm
- net Net-(D3-K): track 6.14 -> 0.00 mm
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- removed copper zone on F.Cu, net /CSN1
- removed copper zone on F.Cu, net /CSP2
- removed copper zone on F.Cu, net /LX1
- removed copper zone on F.Cu, net /LX2
- removed copper zone on F.Cu, net VIN
- removed copper zone on F.Cu, net VOUT
Other:
- board text removed: "PGOOD"
- board text removed: "VCC"
